Commit message: 添加io控制

File: hsr_irp_jr603/hsr_description/urdf/hsr_jr603.urdf (robot description, URDF)
Before this commit: robot hsr_jr603, 8 links, 7 joints
Joints:
- joint joint_6: limit lower=-6.283185307179 upper=6.283185307179 effort=28 velocity=3.2 -> lower=-3.141593 upper=3.141593 effort=28 velocity=3.2

Commit message: 调试ing

File: hsr_irp_jr603/hsr_description/urdf/hsr_jr603.urdf (robot description, URDF)
Before this commit: robot hsr_jr603, 8 links, 7 joints
Joints:
- joint joint_1: limit lower=-3.1415 upper=3.1415 effort=28 velocity=3.2 -> lower=-2.93 upper=2.93 effort=28 velocity=3.2
- joint joint_2: limit lower=-2.7038 upper=0.08722 effort=28 velocity=3.2 -> lower=-2.7038 upper=0 effort=28 velocity=3.2
- joint joint_3: limit lower=-0.349 upper=4.1015 effort=28 velocity=3.2 -> lower=-0.14 upper=4.1 effort=28 velocity=3.2
- joint joint_4: limit lower=-3.124139 upper=3.124139 effort=28 velocity=3.2 -> lower=-2.72 upper=2.72 effort=28 velocity=3.2
